File: bm1370.kicad_sch (KiCad schematic)
At the start: 49 parts, among them U5 MCP1824T-1202E/OT, U6 MCP1824T-0802E, U7 25MHz, U8 BM1370_mode1, U9 SN74AVC4T774

Commit message: bump to 602
Parts:
- added R20, R26: R_US, Resistor_SMD:R_0402_1005Metric, symbol Device:R_US
- renumbered R6 to R17, R6 to R18, R6 to R19
Connections:
- net 0V8: now also C45.1, U8.17 (VDDIO_08_1), R26.1
- net 1V2: now also C42.1, U8.16 (VDDIO_12_1), R20.1
- net at U6.4 (PG): now also R26.2
- net at U5.4 (PG): now also R20.2
- no-connect marks 3 -> 1
Other:
- moved on the sheet: C26, C27
