File: esp32.kicad_sch (KiCad schematic)
At the start: 21 parts, among them J2 TC2030-IDC, J3 Conn_01x04, J4 Conn_01x06, J5 USB_C_Receptacle_USB2.0, SW1 GT-TC029B-H025-L1N, SW2 GT-TC029B-H025-L1N, U3 RT9080-33GJ5, U4 ESP32-S3-WROOM-1

Commit message: bump to 602
Parts:
- added R27: R_US, Resistor_SMD:R_0402_1005Metric, symbol Device:R_US
- U3: footprint bitaxe:RT9080-33GJ5 -> TSOT-23-5_RIT
Connections:
- net 3V3: now also R27.2
- net at U3.4 (NC): now also R27.1
