File: fan.kicad_sch (KiCad schematic)
At the start: 14 parts, among them J6 Conn_01x04, U10 EMC2101

Commit message: bump to 602
Parts:
- renumbered R51 to R24
Changed lines of the file:
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@@
 (kicad_sch
-	(version 20231120)
+	(version 20250114)
 	(generator "eeschema")
-	(generator_version "8.0")
+	(generator_version "9.0")
 	(paper "A")
 	(title_block
@@
 		(rev "600")
 	)
+	(text "EMC2101 Controls the fan, and reads the ASIC chip temperature"
+		(exclude_from_sim no)
+		(at 114.3 63.5 0)
+		(effects
+			(font
+				(size 1.27 1.27)
+			)
+			(justify left bottom)
+		)
+	)
+	(text "This sets default fan speed to 100% ->"
+		(exclude_from_sim no)
+		(at 105.41 106.68 0)
+		(effects
+			(font
+				(size 1.27 1.27)
+			)
+			(justify left bottom)
+		)
+	)
+	(text "I2C Address: 0x4C"
+		(exclude_from_sim no)
+		(at 137.16 90.17 0)
+		(effects
+			(font
+				(size 1.27 1.27)
+			)
+			(justify left bottom)
+		)
+	)
 	(junction
 		(at 82.55 73.66)
@@
 		)
 	)
-	(text "EMC2101 Controls the fan, and reads the ASIC chip temperature"
-		(exclude_from_sim no)
-		(at 114.3 63.5 0)
-		(effects
-			(font
-				(size 1.27 1.27)
-			)
-			(justify left bottom)
-		)
-	)
-	(text "This sets default fan speed to 100% ->"
-		(exclude_from_sim no)
-		(at 105.41 106.68 0)
-		(effects
-			(font
-				(size 1.27 1.27)
-			)
-			(justify left bottom)
-		)
-	)
-	(text "I2C Address: 0x4C"
-		(exclude_from_sim no)
-		(at 137.16 90.17 0)
-		(effects
-			(font
-				(size 1.27 1.27)
-			)
-			(justify left bottom)
-		)
-	)
 	(label "5V"
 		(at 184.15 66.04 0)
-		(fields_autoplaced yes)
 		(effects
 			(font
@@
 	(label "FAN_PWM"
 		(at 160.02 78.74 0)
-		(fields_autoplaced yes)
 		(effects
 			(font
@@
 	(label "TEMP_DN"
 		(at 120.65 81.28 0)
-		(fields_autoplaced yes)
 		(effects
 			(font
@@
 	(label "GND"
 		(at 160.02 83.82 0)
-		(fields_autoplaced yes)
 		(effects
 			(font
@@
 	(label "TEMP_P"
 		(at 73.66 73.66 0)
-		(fields_autoplaced yes)
 		(effects
 			(font
@@
 	(label "SCL"
 		(at 165.1 73.66 0)
-		(fields_autoplaced yes)
 		(effects
 			(font
@@
 	(label "3V3"
 		(at 147.32 101.6 0)
-		(fields_autoplaced yes)
 		(effects
 			(font
@@
 	(label "FAN_TACH"
 		(at 120.65 83.82 0)
-		(fields_autoplaced yes)
 		(effects
 			(font
@@
 	(label "GND"
 		(at 157.48 127 0)
-		(fields_autoplaced yes)
 		(effects
 			(font
@@
 	(label "FAN_PWM"
 		(at 168.91 109.22 0)
-		(fields_autoplaced yes)
 		(effects
 			(font
@@
 	(label "3V3"
 		(at 125.73 73.66 0)
-		(fields_autoplaced yes)
 		(effects
 			(font
@@
 	(label "5V"
 		(at 138.43 114.3 0)
-		(fields_autoplaced yes)
 		(effects
 			(font
@@
 	(label "SDA"
 		(at 165.1 76.2 0)
-		(fields_autoplaced yes)
 		(effects
 			(font
@@
 	(label "TEMP_DP"
 		(at 120.65 78.74 0)
-		(fields_autoplaced yes)
 		(effects
 			(font
@@
 	(label "TEMP_N"
 		(at 73.66 76.2 0)
-		(fields_autoplaced yes)
 		(effects
 			(font
@@
 	(label "FAN_TACH"
 		(at 168.91 111.76 0)
-		(fields_autoplaced yes)
 		(effects
 			(font
@@
 		(shape input)
 		(at 135.89 114.3 180)
-		(fields_autoplaced yes)
 		(effects
 			(font
@@
 		(shape input)
 		(at 73.66 73.66 180)
-		(fields_autoplaced yes)
 		(effects
 			(font
@@
 		(shape input)
 		(at 73.66 76.2 180)
-		(fields_autoplaced yes)
 		(effects
 			(font
@@
 		(shape input)
 		(at 171.45 73.66 0)
-		(fields_autoplaced yes)
 		(effects
 			(font
@@
 		(shape input)
 		(at 125.73 73.66 180)
-		(fields_autoplaced yes)
 		(effects
 			(font
@@
 		(shape input)
 		(at 171.45 76.2 0)
-		(fields_autoplaced yes)
 		(effects
 			(font
@@
 		(on_board yes)
 		(dnp no)
-		(property "Reference" "R51"
+		(property "Reference" "R24"
 			(at 151.13 105.41 0)
 			(effects
@@
 			)
 		)
-		(property "Description" ""
+		(property "Description" "C227158"
 			(at 147.32 106.68 0)
 			(effects
@@
 			)
 		)
-		(property "Description" ""
+		(property "Description" "C1525"
 			(at 191.77 77.47 0)
 			(effects
@@
 			)
 		)
-		(property "Description" ""
+		(property "Description" "C1525"
 			(at 151.13 119.38 0)
 			(effects
@@
 			)
 		)
-		(property "Description" ""
+		(property "Description" "C138288"
 			(at 90.17 76.2 0)
 			(effects
@@
 			)
 		)
-		(property "Description" ""
+		(property "Description" "C272887"
 			(at 106.68 80.01 0)
 			(effects
@@
 			)
 		)
-		(property "Description" ""
+		(property "Description" "C2932477"
 			(at 144.78 119.38 0)
 			(effects
@@
 			)
 		)
-		(property "Description" ""
+		(property "Description" "C240840"
 			(at 184.15 114.3 0)
 			(effects
@@
 			)
 		)
-		(property "Description" ""
+		(property "Description" "C138288"
 			(at 91.44 73.66 0)
 			(effects
@@
 			)
 		)
-		(property "Description" ""
+		(property "Description" "C190095"
 			(at 179.07 72.39 0)
 			(effects
@@
 			)
 		)
-		(property "Description" ""
+		(property "Description" "C626968"
 			(at 144.78 78.74 0)
 			(effects
